File: led_strip_scriptout.kicad_pcb (KiCad board)
At the start: 2 copper layers, 895.4 x 12.7 mm, 1339 parts

Commit message: Schematic and layout complete. Just need to work on getting the BOM in a good format
Parts:
- removed REF** (x58): via-20mil, vias:via-20mil
- removed REF** (x2): pad-50mil, vias:pad-60mil
- added R1760: 0, Resistors_SMD:R_0805, B.Cu at (-39.1, 141.1)
- moved R1758 66.4 mm to (-36.3, 136.9)
- moved R1748 66.3 mm to (-16.8, 141.1)
- moved R1759 66.3 mm to (-36.3, 145.3)
- moved R1757 66.3 mm to (-33.5, 141.1)
- moved R1749 66.3 mm to (-19.6, 136.9)
- moved D1701 66.3 mm to (69.8, 141.0)
- moved D1702 66.3 mm to (64.2, 141.0)
- moved D1703 66.3 mm to (58.7, 141.0)
- moved D1704 66.3 mm to (53.1, 141.0)
- moved D1705 66.3 mm to (47.5, 141.0)
- moved D1706 66.3 mm to (41.9, 141.0)
- moved D1707 66.3 mm to (36.3, 141.0)
- moved D1708 66.3 mm to (30.7, 141.0)
- moved D1709 66.3 mm to (25.1, 141.0)
- moved D1710 66.3 mm to (19.5, 141.0)
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Connections:
- net /LastBlock/IN renamed /Block16/IN
- R1046 pad 1: Net-(R1046-Pad1) -> VDD
- R1146 pad 1: Net-(R1146-Pad1) -> VDD
- R1246 pad 1: Net-(R1246-Pad1) -> VDD
- R1346 pad 1: Net-(R1346-Pad1) -> VDD
- R1446 pad 1: Net-(R1446-Pad1) -> VDD
- R1546 pad 1: Net-(R1546-Pad1) -> VDD
- R1646 pad 1: Net-(R1646-Pad1) -> VDD
- R246 pad 1: Net-(R246-Pad1) -> VDD
- R346 pad 1: Net-(R346-Pad1) -> VDD
- R446 pad 1: Net-(R446-Pad1) -> VDD
- R546 pad 1: Net-(R546-Pad1) -> VDD
- R646 pad 1: Net-(R646-Pad1) -> VDD
- R746 pad 1: Net-(R746-Pad1) -> VDD
- R846 pad 1: Net-(R846-Pad1) -> VDD
- R946 pad 1: Net-(R946-Pad1) -> VDD
- R960 pad 1: /Block9/IN -> /Block8/OUT
Routing:
- net Net-(D1001-Pad1): track 5.84 -> 46.7 mm
- net Net-(D1002-Pad2): track 5.22 -> 41.7 mm
- net Net-(D1003-Pad1): track 5.20 -> 41.6 mm
- net Net-(D1007-Pad1): track 5.20 -> 41.6 mm
- net Net-(D1004-Pad1): track 5.20 -> 41.6 mm
- net Net-(D1006-Pad1): track 5.20 -> 41.6 mm
- net Net-(D1005-Pad1): track 5.20 -> 41.6 mm
- net Net-(D1008-Pad1): track 5.20 -> 41.6 mm
- net Net-(D1002-Pad1): track 5.20 -> 41.6 mm
- net Net-(D1017-Pad2): track 5.07 -> 40.6 mm
- net Net-(D1013-Pad1): track 5.07 -> 40.6 mm
- net Net-(D1020-Pad2): track 5.07 -> 40.6 mm
- net Net-(D1010-Pad2): track 5.07 -> 40.6 mm
- net Net-(D1019-Pad1): track 5.07 -> 40.6 mm
- net Net-(D1014-Pad1): track 5.07 -> 40.6 mm
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- removed copper zone on B.Cu, net GND
- removed copper zone on F.Cu, net GND
- removed copper zone on B.Cu, net VDD
- removed copper zone on F.Cu, net VDD
Other:
- board size 895.4 x 12.7 mm -> 885.2 x 12.7 mm
- board text removed: "0.062 in (nominal)"
- board text removed: "1 oz copper"
- board text removed: "FR4 core"
- board text removed: "GND"
- board text removed: "VDD"
